File: hardware/carrier/pcb/carrier.kicad_pcb (KiCad board)
At the start: 2 copper layers, 65 x 58.5 mm, 91 parts, among them J1 Kit 1-10, J10 ISM330, J11 Cue L, J12 Cue R, J13 Harness M8, J2 Kit 11-20, J3 Kit 40-31, J4 Kit 30-21, J5 Kit J2 feed, J6 Panels A/GND/B, J7 Qwiic spare, J8 M10S J5, J9 M10S J3, U1 BQ24074RGT, U2 TCA4307, U3 TPS2553, U4 USBLC6-2SC6, U5 USBLC6-2SC6

Commit message: Carrier rev A3: fuel gauge, flash, reverse protection; fix socket footprints
Adds the MAX17260 fuel gauge (high-side, 10 mOhm Kelvin sense), W25Q128JV
flash on the spare GPIOs, and AO3401A reverse-battery protection; charger
resistors move to JLCPCB basic values. The plug-in sockets switch to
Pin1Right: JLCPCB's own footprints for the hanxia sockets are the mirror
of Pin1Left, so A2 couldn't have been assembled.

finish_routing.py now brings Inky's board up to the schematic and routes
what changed with Freerouting plus a grid router with rip-up. KiCad DRC at
every severity: 0 violations, 0 unconnected. New: fit_test.py (1:1 paper
fit test) and jlc_files.py (BOM and placement from JLCPCB's footprints).

Co-Authored-By: Claude Opus 5.5 (1M context) <noreply@anthropic.com>
Parts:
- added C10: 470n, C_0603_1608Metric, F.Cu at (162.2, 111.2)
- added C11: 100n, C_0603_1608Metric, F.Cu at (159.8, 121.3)
- added C12: 100n, C_0603_1608Metric, F.Cu at (141.5, 123.3)
- added Q1: AO3401A, SOT-23, F.Cu at (161.8, 125.0)
- added R24: 10m, R_0805_2012Metric, F.Cu at (161.8, 121.3)
- added R25: 100k, R_0603_1608Metric, F.Cu at (160.0, 110.9)
- added R26: 100k, R_0603_1608Metric, F.Cu at (141.5, 126.6)
- added U6: MAX17260, TDFN-14-1EP_3x3mm_P0.4mm_EP1.78x2.35mm, F.Cu at (161.8, 115.0)
- added U7: W25Q128JVS, SOIC-8_5.3x5.3mm_P1.27mm, F.Cu at (136.0, 125.0)
- J1, J2, J3, J4: footprint PinSocket_1x10_P2.54mm_Vertical_SMD_Pin1Left -> PinSocket_1x10_P2.54mm_Vertical_SMD_Pin1Right
- J10: footprint PinSocket_1x09_P2.54mm_Vertical_SMD_Pin1Left -> PinSocket_1x09_P2.54mm_Vertical_SMD_Pin1Right
- J8: footprint PinSocket_1x08_P2.54mm_Vertical_SMD_Pin1Left -> PinSocket_1x08_P2.54mm_Vertical_SMD_Pin1Right
- J9: footprint PinSocket_1x04_P2.54mm_Vertical_SMD_Pin1Left -> PinSocket_1x04_P2.54mm_Vertical_SMD_Pin1Right
- R2: value 887 -> 1k
- R3: value 3.24k -> 4.7k
- R4: value 71.5k -> 68k
- moved R5 8.61 mm to (147.9, 115.9), turned to 180 degrees
Connections:
- J1 pad 10: (no net) -> FLASH_CS
- J13 pad 2: BAT -> BAT_PACK
- J13 pad 8: BAT -> BAT_PACK
- J2 pad 1: (no net) -> FLASH_SCK
- J2 pad 2: (no net) -> FLASH_MOSI
- J2 pad 3: (no net) -> FLASH_MISO
- J2 pad 4: (no net) -> FG_ALRT
Routing:
- net GND: track 260.6 -> 43.1 mm, vias 77 -> 140
- net FG_ALRT: track 0.00 -> 105.2 mm, vias 0 -> 2
- net SOLAR_A: track 78.4 -> 163.8 mm, vias 3 -> 15
- net RESET: track 106.8 -> 35.7 mm, vias 13 -> 1
- net I2C_SCL: track 109.1 -> 169.9 mm, vias 5 -> 10
- net FLASH_SCK: track 0.00 -> 47.3 mm, vias 0 -> 8
- net FLASH_CS: track 0.00 -> 45.8 mm
- net FLASH_MOSI: track 0.00 -> 43.5 mm
- net FLASH_MISO: track 0.00 -> 40.7 mm, vias 0 -> 4
- net 3V3: track 200.2 -> 239.1 mm, vias 12 -> 14
- net BAT_PACK: track 0.00 -> 33.9 mm, vias 0 -> 2
- net I2C_SDA: track 124.6 -> 150.4 mm, vias 8 -> 7
- net EXT_SCL: track 164.8 -> 139.5 mm, vias 7 -> 11
- net EXT_3V3: track 134.3 -> 158.4 mm, vias 6 -> 9
- net CHG_STAT: track 53.2 -> 76.9 mm, vias 6 -> 4
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Other:
- board text added: "OpenCollar carrier rev A3"
- board text removed: "OpenCollar carrier rev A2"

Commit message: Add licences: Apache-2.0 code, CERN-OHL-W-2.0 hardware, CC BY 4.0 docs
Adds LICENSE, LICENSES/, NOTICE (names and logo not licensed) and
CONTRIBUTING.md (contributions licensed like the files they touch, with
a relicensing grant to openpasture). Hardware moves from the planned
CERN-OHL-P to CERN-OHL-W; carrier silkscreen text updated, DRC still clean.

Co-Authored-By: Claude Opus 5.5 (1M context) <noreply@anthropic.com>
Other:
- board text added: "CERN-OHL-W 2026-09-27"
- board text removed: "CERN-OHL-P 2026-09-27"
Changed lines of the file:
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@@
 		)
 	)
-	(gr_text "CERN-OHL-P  2026-09-27"
+	(gr_text "CERN-OHL-W  2026-09-27"
 		(at 138 135.3 0)
 		(layer "B.SilkS")
