File: hardware/carrier/pcb/heypcb/opencollar-carrier.kicad_pcb (KiCad board)
At the start: 2 copper layers, 65 x 58.5 mm, 91 parts, among them J1 Kit 1-10, J10 ISM330, J11 Cue L, J12 Cue R, J13 Harness M8, J2 Kit 11-20, J3 Kit 40-31, J4 Kit 30-21, J5 Kit J2 feed, J6 Panels A/GND/B, J7 Qwiic spare, J8 M10S J5, J9 M10S J3, U1 BQ24074RGT, U2 TCA4307, U3 TPS2553, U4 USBLC6-2SC6, U5 USBLC6-2SC6

Commit message: Add licences: Apache-2.0 code, CERN-OHL-W-2.0 hardware, CC BY 4.0 docs
Adds LICENSE, LICENSES/, NOTICE (names and logo not licensed) and
CONTRIBUTING.md (contributions licensed like the files they touch, with
a relicensing grant to openpasture). Hardware moves from the planned
CERN-OHL-P to CERN-OHL-W; carrier silkscreen text updated, DRC still clean.

Co-Authored-By: Claude Opus 5.5 (1M context) <noreply@anthropic.com>
Other:
- board text added: "CERN-OHL-W 2026-09-27"
- board text removed: "CERN-OHL-P 2026-09-27"
Changed lines of the file:
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@@
 		)
 	)
-	(gr_text "CERN-OHL-P  2026-09-27"
+	(gr_text "CERN-OHL-W  2026-09-27"
 		(at 138 135.3 0)
 		(layer "B.SilkS")
